File: MarvinHardware/MarvinKiCad/MarvinKiCad.kicad_sch (KiCad schematic)
At the start: 6 parts

Commit message: worked on schematic and layout
Parts:
- R1, R2, R3: footprint (none) -> Resistor_SMD:R_0402_1005Metric_Pad0.72x0.64mm_HandSolder
Connections:
- new net: R3.2, U1., U2.
- new net: R2.1, U1., U2.
- new net: R1.2, U1., U2.
- new net: U1., U2. (x3)
Changed lines of the file:
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@@
 			)
 		)
-		(property "Footprint" ""
+		(property "Footprint" "Resistor_SMD:R_0402_1005Metric_Pad0.72x0.64mm_HandSolder"
 			(at 73.152 69.85 90)
 			(effects
@@
 			)
 		)
-		(property "Footprint" ""
+		(property "Footprint" "Resistor_SMD:R_0402_1005Metric_Pad0.72x0.64mm_HandSolder"
 			(at 71.628 69.85 90)
 			(effects
@@
 			)
 		)
-		(property "Footprint" ""
+		(property "Footprint" "Resistor_SMD:R_0402_1005Metric_Pad0.72x0.64mm_HandSolder"
 			(at 62.992 69.85 90)
 			(effects
