File: 6_Semester/MarvinHW/KiCad/MarvinProjekt/MarvinProjekt.kicad_pcb (KiCad board)
At the start: 4 copper layers, 73.1 x 86.8 mm, 128 parts, among them J1 Conn_02x03_Odd_Even, J2 Conn_01x04_Pin, Q1 Q_PNP_Darlington_BCE, Q2 Q_PNP_Darlington_BCE, Q3 BC817-40, SW1 Reset, SW2 Boot, SW3 Volume+, SW4 Volume-, SW5 Modi1, SW6 Modi0, SW7 Switch Slide SPDT 100mA 12V, SW8 Reset, SW9 Boot, U1 ESP32-S3-WROOM-1, U10 ToF, U2 ES8388, U3 MP1720, U4 TF_CARD, U5 DW01A, U6 FS8205A, U7 HM4056H, U8 TPLP5907MFX-3.3, U9 WS2812, X1 USB3.1C16PFSMT

Commit message: Finished Layout
Parts:
- added C41: 100nF, Capacitor_SMD:C_0805_2012Metric_Pad1.18x1.45mm_HandSolder, F.Cu at (99.8, 106.8)
- added C42: 100nF, Capacitor_SMD:C_0805_2012Metric_Pad1.18x1.45mm_HandSolder, F.Cu at (102.3, 138.9)
- added C43: 100nF, Capacitor_SMD:C_0805_2012Metric_Pad1.18x1.45mm_HandSolder, F.Cu at (154.8, 139.0)
- added C44: 100nF, Capacitor_SMD:C_0805_2012Metric_Pad1.18x1.45mm_HandSolder, F.Cu at (154.8, 109.2)
- added G***: LOGO, Library:Marivin_liegend, F.Cu at (96.3, 95.5)
- added G***: LOGO, Library:Marvin, B.Cu at (111.9, 134.1)
- added U11: WS2812, LED_SMD:LED_WS2812B-2020_PLCC4_2.0x2.0mm, F.Cu at (102.5, 136.5)
- added U12: WS2812, LED_SMD:LED_WS2812B-2020_PLCC4_2.0x2.0mm, F.Cu at (154.8, 136.6)
- added U13: WS2812, LED_SMD:LED_WS2812B-2020_PLCC4_2.0x2.0mm, F.Cu at (154.8, 106.8)
- moved R35 54.6 mm to (140.3, 99.7)
- moved D1 54.4 mm to (146.2, 98.4)
- moved R1 54.4 mm to (149.4, 94.1)
- moved R34 54.1 mm to (134.8, 96.8), turned to 180 degrees
- moved X1 53.7 mm to (156.7, 99.5)
- moved R2 52.6 mm to (146.3, 104.1)
- moved D4 51.2 mm to (157.5, 92.9)
- moved R38 51.2 mm to (153.8, 92.9)
- moved D5 51.1 mm to (157.4, 90.9)
- moved R41 51.1 mm to (153.7, 91.0)
- moved C1 50.7 mm to (148.7, 102.1), turned to 180 degrees
- moved U6 50.5 mm to (136.7, 103.6), turned to 0 degrees
- moved U5 48.7 mm to (137.1, 99.7), turned to 180 degrees
- moved C35 47.3 mm to (133.9, 99.7), turned to -90 degrees
- moved C36 44.1 mm to (138.1, 106.7)
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Connections:
- U1 pad 17: BATTERY_CHRG_EANBLE -> BAT_FB
- U1 pad 18: BAT_FB -> ENABLE_BATTERY_CHRG
- U1 pad 19: MODI1 -> VOLUME-
- U1 pad 20: MODI2 -> VOLUME+
- U1 pad 21: VOLUME+ -> MODI2
- U1 pad 22: VOLUME- -> MODI1
- U9 pad 1: unconnected-(U9-DOUT-Pad1) -> Net-(U11-DIN)
Routing:
- net +3.3V: track 0.00 -> 217.3 mm, vias 0 -> 8
- net V_Audio: track 0.00 -> 155.6 mm, vias 0 -> 6
- net V_LED: track 0.00 -> 155.1 mm, vias 0 -> 7
- net GND: track 0.00 -> 130.2 mm, vias 0 -> 86
- net ESP_GPIO0: track 0.00 -> 101.4 mm, vias 0 -> 6
- net SDA: track 0.00 -> 85.9 mm, vias 0 -> 2
- net Net-(BT1--): track 0.00 -> 85.8 mm, vias 0 -> 3
- net SCL: track 0.00 -> 85.6 mm, vias 0 -> 2
- net V_Bat: track 0.00 -> 83.9 mm, vias 0 -> 1
- net ESP_EN: track 0.00 -> 80.3 mm, vias 0 -> 4
- net MODI2: track 0.00 -> 68.7 mm, vias 0 -> 4
- net ESP_U0_TX: track 0.00 -> 66.6 mm, vias 0 -> 2
- net ESP_U0_RX: track 0.00 -> 66.3 mm, vias 0 -> 3
- net V_Audio_ENABLE: track 0.00 -> 64.3 mm, vias 0 -> 2
- net IO02: track 0.00 -> 60.7 mm, vias 0 -> 1
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