File: 6_Semester/MarvinHW/KiCad/MarvinProjekt/MarvinProjekt.kicad_pcb (KiCad board)
At the start: 4 copper layers, 73.1 x 86.8 mm, 137 parts, among them J1 Conn_02x03_Odd_Even, J2 Conn_01x04_Pin, Q1 Q_PNP_Darlington_BCE, Q2 Q_PNP_Darlington_BCE, Q3 BC817-40, SW1 Reset, SW2 Boot, SW3 Volume+, SW4 Volume-, SW5 Modi1, SW6 Modi0, SW7 Switch Slide SPDT 100mA 12V, SW8 Reset, SW9 Boot, U1 ESP32-S3-WROOM-1, U10 ToF, U11 WS2812, U12 WS2812, U13 WS2812, U2 ES8388, U3 MP1720, U4 TF_CARD, U5 DW01A, U6 FS8205A, U7 HM4056H, U8 TPLP5907MFX-3.3, U9 WS2812, X1 USB3.1C16PFSMT

Commit message: creat new grb files
Other:
- board text added: "Marvin"
- board text added: "Nora Hüppi"
- board text added: "V 2.0"
