File: 6_Semester/MarvinHW/KiCad/MarvinProjekt/MarvinProjekt.kicad_sch (KiCad schematic)
At the start: 37 parts, among them J1 Conn_02x03_Odd_Even, J2 Conn_01x04_Pin, SW1 Reset, SW2 Boot, SW3 Volume+, SW4 Volume-, SW5 Modi1, SW6 Modi0, SW8 Reset, SW9 Boot, U1 ESP32-S3-WROOM-1, U10 ToF, U11 WS2812, U12 WS2812, U13 WS2812, U9 WS2812, X1 USB3.1C16PFSMT

Commit message: finish evaluat components
Parts:
- U10: now not fitted
Changed lines of the file:
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@@
 		(in_bom yes)
 		(on_board yes)
-		(dnp no)
+		(dnp yes)
 		(fields_autoplaced yes)
 		(property "Reference" "U10"
