File: 6_Semester/MarvinHW/KiCad/MarvinProjekt/Power.kicad_sch (KiCad schematic)
At the start: 14 parts, among them Q1 Q_PNP_Darlington_BCE, Q2 Q_PNP_Darlington_BCE, Q3 BC817-40, SW7 Switch Slide SPDT 100mA 12V, U8 TPLP5907MFX-3.3

Commit message: add comonents to BoM
Parts:
- Q1, Q2: OrderNow (none) -> x
- U8: LCSC Part (none) -> C460335; OrderNow (none) -> x
Changed lines of the file:
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@@
 			)
 		)
-		(property "Datasheet" "file:///C:/data/Schule/BuP/5_Semester/Marvin/MarvinProject/6_Semester/MarvinDatenblaetter/LinearVoltageRegulator/2411121130_TECH-PUBLIC-TPLP5907MFX-3-3_C5370990.pdf"
+		(property "Datasheet" "file:///C:/data/Schule/BuP/5_Semester/Marvin/MarvinProject/6_Semester/MarvinDatenblaetter/LinearVoltageRegulator/AP2138-9.pdf"
 			(at 63.5 34.29 0)
 			(effects
@@
 			)
 		)
+		(property "OrderNow" "x"
+			(at 63.5 34.29 0)
+			(effects
+				(font
+					(size 1.27 1.27)
+				)
+				(hide yes)
+			)
+		)
+		(property "LCSC Part" "C460335"
+			(at 63.5 34.29 0)
+			(effects
+				(font
+					(size 1.27 1.27)
+				)
+				(hide yes)
+			)
+		)
 		(pin "4"
 		)
@@
 		)
 		(property "Sim.Pins" "1=C 2=B 3=E"
+			(at 57.15 138.43 0)
+			(effects
+				(font
+					(size 1.27 1.27)
+				)
+				(hide yes)
+			)
+		)
+		(property "OrderNow" ""
 			(at 57.15 138.43 0)
 			(effects
@@
 			)
 		)
+		(property "OrderNow" "x"
+			(at 55.88 64.77 0)
+			(effects
+				(font
+					(size 1.27 1.27)
+				)
+				(hide yes)
+			)
+		)
 		(pin "1"
 		)
@@
 			)
 		)
+		(property "OrderNow" ""
+			(at 52.07 120.65 0)
+			(effects
+				(font
+					(size 1.27 1.27)
+				)
+				(hide yes)
+			)
+		)
 		(pin "1"
 		)
@@
 		)
 		(property "Description" "Resistor"
+			(at 59.69 127 0)
+			(effects
+				(font
+					(size 1.27 1.27)
+				)
+				(hide yes)
+			)
+		)
+		(property "OrderNow" ""
 			(at 59.69 127 0)
 			(effects
@@
 			)
 		)
+		(property "OrderNow" ""
+			(at 29.21 27.94 0)
+			(effects
+				(font
+					(size 1.27 1.27)
+				)
+				(hide yes)
+			)
+		)
 		(pin "3"
 		)
@@
 			)
 		)
+		(property "OrderNow" "x"
+			(at 59.69 113.03 0)
+			(effects
+				(font
+					(size 1.27 1.27)
+				)
+				(hide yes)
+			)
+		)
 		(pin "1"
 		)
@@
 			)
 		)
+		(property "OrderNow" ""
+			(at 46.99 36.83 0)
+			(effects
+				(font
+					(size 1.27 1.27)
+				)
+				(hide yes)
+			)
+		)
 		(pin "2"
 		)
@@
 			)
 		)
+		(property "OrderNow" ""
+			(at 39.37 36.83 0)
+			(effects
+				(font
+					(size 1.27 1.27)
+				)
+				(hide yes)
+			)
+		)
 		(pin "2"
 		)
@@
 			)
 		)
+		(property "OrderNow" ""
+			(at 44.45 138.43 0)
+			(effects
+				(font
+					(size 1.27 1.27)
+				)
+				(hide yes)
+			)
+		)
 		(pin "1"
 		)
@@
 		)
 		(property "Description" "Resistor"
+			(at 52.07 69.85 0)
+			(effects
+				(font
+					(size 1.27 1.27)
+				)
+				(hide yes)
+			)
+		)
+		(property "OrderNow" ""
 			(at 52.07 69.85 0)
 			(effects
@@
 			)
 		)
+		(property "OrderNow" ""
+			(at 87.63 36.83 0)
+			(effects
+				(font
+					(size 1.27 1.27)
+				)
+				(hide yes)
+			)
+		)
 		(pin "2"
 		)
@@
 		)
 		(property "Description" "Unpolarized capacitor"
+			(at 80.01 36.83 0)
+			(effects
+				(font
+					(size 1.27 1.27)
+				)
+				(hide yes)
+			)
+		)
+		(property "OrderNow" ""
 			(at 80.01 36.83 0)
 			(effects
@@
 			(at 55.88 76.2 0)
 			(effects
+				(font
+					(size 1.27 1.27)
+				)
+				(hide yes)
+			)
+		)
+		(property "OrderNow" ""
+			(at 55.88 76.2 0)
+			(effects

Commit message: finish evaluat components
Parts:
- Q1, Q2: LCSC Part (none) -> C130420
Changed lines of the file:
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@@
+			)
+		)
+		(property "LCSC Part" "C130420"
+			(at 55.88 64.77 0)
+			(effects
+				(font
+					(size 1.27 1.27)
+				)
+				(hide yes)
 			)
 		)
@@
 			(at 59.69 113.03 0)
 			(effects
+				(font
+					(size 1.27 1.27)
+				)
+				(hide yes)
+			)
+		)
+		(property "LCSC Part" "C130420"
+			(at 59.69 113.03 0)
+			(effects
